File: padrino-328p.kicad_pcb (KiCad board)
At the start: 2 copper layers, 68.6 x 53.3 mm, 56 parts, among them J1 CONN_01X03, P1 CONN_01X08, P2 CONN_01X10, P3 CONN_01X06, P4 CONN_01X08, P5 ICSP, P6 USB_OTG, P7 BARREL_JACK, Q1 MOSFET_P, SW1 CONN_01X02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

Commit message: Arregladas orientación del botón de reset y pinout del regulador de 3.3V
Parts:
- moved SW1 2.50 mm to (165.1, 136.4), turned to 90 degrees
Routing:
- net /RESET: track 81.7 -> 87.2 mm
- net GNDREF: track 316.0 -> 318.5 mm
- net +3V3: track 65.0 -> 66.2 mm
Other:
- board text added: "Diseñado en España Ensamblado en la UE FABRICADIGITAL.ORG"
- board text removed: "Diseñada en España Ensamblada en la UE FABRICADIGITAL.ORG"
